File: Schematic/YM2612_MIDI_SMD/YM2612_MIDI_SMD.sch (KiCad schematic (older format))
At the start: 122 parts, among them J1 Barrel_Jack_12V, J2 USB_B, J3 DIN-5_180, J4 Audio-Jack-3, J5 Micro_SD_Card, J6 ICSP, J7 TP_GND, SW1 SW_Push_Dual, SW10 SW_Push_Dual, SW2 SW_Push_Dual, SW3 SW_Push_Dual, SW4 SW_Push_Dual, SW5 SW_Push_Dual, SW6 SW_Push_Dual, SW7 SW_Push_Dual, SW8 SW_Push_Dual, SW9 Rotary_Encoder_Switch, U1 LM2596S-5, U10 LD1117S33TR_SOT223, U11 4050, U2 AT90USB1286-AU, U3 YM2612, U4 SN76489, U6 H11L1, U8 TPA3122D2, U9 TL062, Y1 16MHz

Commit message: Fixed minor bug on favorite button #7
Parts:
- J5: footprint Connector_Card:microSD_HC_Hirose_DM3D-SF -> customMicroSD:SOFNG_TF_15x15_PUSH_PUSH
- U6: footprint Housings_DIP:DIP-6_W7.62mm -> Housings_DIP:SMDIP-6_W7.62mm
Changed lines of the file:
@@
 F 0 "U6" H 2500 10050 50  0000 L CNN
 F 1 "H11L1" H 2500 9950 50  0000 L CNN
-F 2 "Housings_DIP:DIP-6_W7.62mm" H 2210 10150 50  0001 C CNN
+F 2 "Housings_DIP:SMDIP-6_W7.62mm" H 2210 10150 50  0001 C CNN
 F 3 "https://www.fairchildsemi.com/datasheets/H1/H11L1M.pdf" H 2210 10150 50  0001 C CNN
 	1    2300 10150
@@
 F 0 "J5" H 14700 7667 50  0000 C CNN
 F 1 "Micro_SD_Card" H 14700 7576 50  0000 C CNN
-F 2 "Connector_Card:microSD_HC_Hirose_DM3D-SF" H 15900 7250 50  0001 C CNN
+F 2 "customMicroSD:SOFNG_TF_15x15_PUSH_PUSH" H 15900 7250 50  0001 C CNN
 F 3 "http://katalog.we-online.de/em/datasheet/693072010801.pdf" H 14750 6950 50  0001 C CNN
 	1    14750 6950
@@
 	6500 6450 6800 6450
 $Comp
-L power:GND #PWR?
+L power:GND #PWR0112
 U 1 1 5CD1BBF6
 P 7950 2750
-F 0 "#PWR?" H 7950 2500 50  0001 C CNN
+F 0 "#PWR0112" H 7950 2500 50  0001 C CNN
 F 1 "GND" H 7955 2577 50  0000 C CNN
 F 2 "" H 7950 2750 50  0001 C CNN
@@
 	10450 1600 10450 1950
 $Comp
-L power:GND #PWR?
+L power:GND #PWR0113
 U 1 1 5CD2D4AE
 P 10900 2100
-F 0 "#PWR?" H 10900 1850 50  0001 C CNN
+F 0 "#PWR0113" H 10900 1850 50  0001 C CNN
 F 1 "GND" H 10905 1927 50  0000 C CNN
 F 2 "" H 10900 2100 50  0001 C CNN
@@
 $EndComp
 $Comp
-L power:GND #PWR?
+L power:GND #PWR0114
 U 1 1 5CD2D5B9
 P 11200 2000
-F 0 "#PWR?" H 11200 1750 50  0001 C CNN
+F 0 "#PWR0114" H 11200 1750 50  0001 C CNN
 F 1 "GND" H 11205 1827 50  0000 C CNN
 F 2 "" H 11200 2000 50  0001 C CNN
@@
 $EndComp
 $Comp
-L power:GND #PWR?
+L power:GND #PWR0116
 U 1 1 5CD2F8C4
 P 15150 1850
-F 0 "#PWR?" H 15150 1600 50  0001 C CNN
+F 0 "#PWR0116" H 15150 1600 50  0001 C CNN
 F 1 "GND" H 15155 1677 50  0000 C CNN
 F 2 "" H 15150 1850 50  0001 C CNN
@@
 	15150 1800 15150 1850
 $Comp
-L power:GND #PWR?
+L power:GND #PWR0117
 U 1 1 5CD41654
 P 7300 1750
-F 0 "#PWR?" H 7300 1500 50  0001 C CNN
+F 0 "#PWR0117" H 7300 1500 50  0001 C CNN
 F 1 "GND" H 7305 1577 50  0000 C CNN
 F 2 "" H 7300 1750 50  0001 C CNN
@@
 	7100 1750 7300 1750
 $Comp
-L power:GND #PWR?
+L power:GND #PWR0118
 U 1 1 5CD5460A
 P 14750 2550
-F 0 "#PWR?" H 14750 2300 50  0001 C CNN
+F 0 "#PWR0118" H 14750 2300 50  0001 C CNN
 F 1 "GND" H 14755 2377 50  0000 C CNN
 F 2 "" H 14750 2550 50  0001 C CNN

Commit message: LC filter value correction
Parts:
- C31, C32: value 68nF -> 0.68uF
- L3, L4: value 2.2mH -> 22uH
Changed lines of the file:
@@
 P 14100 3650
 F 0 "L3" V 14150 3650 50  0000 C CNN
-F 1 "2.2mH" V 14050 3600 50  0000 C CNN
+F 1 "22uH" V 14050 3600 50  0000 C CNN
 F 2 "Inductors_THT:L_Radial_D8.7mm_P5.00mm_Fastron_07HCP" H 14100 3650 50  0001 C CNN
 F 3 "" H 14100 3650 50  0001 C CNN
@@
 P 14350 3550
 F 0 "C31" H 14442 3596 50  0000 L CNN
-F 1 "68nF" H 14442 3505 50  0000 L CNN
+F 1 "0.68uF" H 14442 3505 50  0000 L CNN
 F 2 "Capacitors_SMD:C_0805" H 14350 3550 50  0001 C CNN
 F 3 "" H 14350 3550 50  0001 C CNN
@@
 P 14150 4350
 F 0 "L4" V 14335 4350 50  0000 C CNN
-F 1 "2.2mH" V 14244 4350 50  0000 C CNN
+F 1 "22uH" V 14244 4350 50  0000 C CNN
 F 2 "Inductors_THT:L_Radial_D8.7mm_P5.00mm_Fastron_07HCP" H 14150 4350 50  0001 C CNN
 F 3 "" H 14150 4350 50  0001 C CNN
@@
 P 14350 4450
 F 0 "C32" H 14442 4496 50  0000 L CNN
-F 1 "68nF" H 14442 4405 50  0000 L CNN
+F 1 "0.68uF" H 14442 4405 50  0000 L CNN
 F 2 "Capacitors_SMD:C_0805" H 14350 4450 50  0001 C CNN
 F 3 "" H 14350 4450 50  0001 C CNN

Commit message: Begin hardware revision. New amp
Parts:
- removed C19: 1000uF, Capacitors_SMD:CP_Elec_10x10, symbol device:CP_Small
- removed C22, C23, C24, C25: 1uF, Capacitors_SMD:C_1206, symbol device:CP1_Small
- removed C26: 68uF, Capacitors_SMD:CP_Elec_6.3x5.8, symbol device:CP1_Small
- removed C27: 100uF, Capacitors_SMD:CP_Elec_6.3x7.7, symbol device:CP1_Small
- removed C28, C29: 0.22uF, Capacitors_SMD:C_0805, symbol device:C_Small
- removed C30: 220pF, Capacitors_SMD:C_0603, symbol device:C_Small
- removed C31, C32: 0.68uF, Capacitors_SMD:C_0805, symbol device:C_Small
- removed C33, C34: 10uF, Capacitors_SMD:C_1206, symbol device:C_Small
- removed C35: 1uF, Capacitors_SMD:C_1206, symbol device:C_Small
- removed C36, C37: 1000uF, Capacitors_SMD:CP_Elec_10x10, symbol device:CP1_Small
- removed C38, C39, C40, C41: 5.6nF, Capacitors_SMD:C_0603, symbol device:C_Small
- removed C42: 100nF, Capacitors_SMD:C_0805, symbol device:C_Small
- removed L3, L4: 22uH, Inductors_THT:L_Radial_D8.7mm_P5.00mm_Fastron_07HCP, symbol device:L_Small
- removed R10, R11: 47k, Resistors_SMD:R_0805, symbol device:R
- removed R12, R13, R14, R15, R16: 2.2k, Resistors_SMD:R_0805, symbol device:R
- removed R17, R18, R23, R24: 33k, Resistors_SMD:R_0805, symbol device:R
- removed R19, R20, R21, R22: 10k, Resistors_SMD:R_0805, symbol device:R
- removed U8: TPA3122D2, Housings_DIP:DIP-20_W7.62mm, symbol TPA3122D2:TPA3122D2
- removed U9: TL062, Housings_SOIC:SOIC-8_3.9x4.9mm_Pitch1.27mm, symbol linear:TL062
- added C10, C15: 10uF, symbol device:C_Small
- added C11, C13: 1uF, symbol device:C_Small
- added C17: 100nF, Capacitors_SMD:C_0805, symbol device:C_Small
- added C19, C21: 270pF, symbol device:C_Small
- added C22, C23, C9: 100uF, symbol device:CP_Small
- added C24: 10uF, symbol device:CP_Small
- added R10, R6, R7: 2.2K, symbol device:R_Small
- added R11, R14: 6.2K, symbol device:R_Small
- added R12, R13: 51K, symbol device:R_Small
- added R15, R16: 160K, symbol device:R_Small
- added R4, R5: 10K, symbol device:R_Small
- added U5: TL072, symbol linear:TL072
Connections:
- net labels added: +2V5, +5VA, GNDA
- net labels removed: AVCC, AVCC_DIV2, PRE_L, PRE_R
- wire segments 246 -> 184
Other:
- moved on the sheet: C14, C20

Commit message: Re-annotate
Parts:
- renumbered C48 to C10, C18 to C11, C20 to C12, C3 to C13, C8 to C15, C44 to C16, C45 to C17, C9 to C18, C10 to C19, C11 to C20, C13 to C21, C15 to C22, C24 to C23, C19 to C24, C21 to C25, C46 to C26, C17 to C27, C47 to C28, C22 to C29, C4 to C3, C23 to C30, C5 to C4, C6 to C5, C7 to C6, C16 to C7, C43 to C8, C12 to C9, D9 to D10, D10 to D11, D11 to D3, D3 to D4, D4 to D5, D5 to D6, D6 to D7, D7 to D8, D8 to D9, J3 to J1, J7 to J2, J2 to J3, J1 to J4, J6 to J5, J4 to J6, J5 to J7, L2 to L1, L1 to L2, R26 to R1, R28 to R10, R29 to R11, R30 to R12, R31 to R13, R32 to R14, R33 to R15, R34 to R16, R35 to R17, R4 to R18, R5 to R19, R8 to R2, R6 to R20, R7 to R21, R10 to R22, R11 to R23, R12 to R24, R13 to R25, R14 to R26, R15 to R27, R16 to R28, R1 to R3, R2 to R4, R3 to R5, R27 to R6, R9 to R7, R25 to R8, R36 to R9, SW9 to SW1, SW8 to SW10, SW1 to SW2, SW5 to SW3, SW2 to SW4, SW6 to SW5, SW3 to SW6, SW10 to SW8, SW4 to SW9, U6 to U1, U1 to U5, U10 to U6, U11 to U7, U5 to U8

Commit message: New power delivery
Parts:
- removed C13, C15: 100uF, Capacitors_SMD:CP_Elec_6.3x7.7, symbol device:CP1_Small
- removed C23: 10uF, symbol device:CP_Small
- removed C9: 1000uF, Capacitors_SMD:CP_Elec_10x10, symbol device:CP_Small
- removed D2: LED_Small, LEDs:LED_0805, symbol device:LED_Small
- removed D3: SS34_SMA, Diodes_SMD:D_SMA, symbol device:D_Schottky_Small_ALT
- removed J4: Barrel_Jack_12V, Connectors:BARREL_JACK, symbol conn:Barrel_Jack
- removed L2: 33uH, custom_inductors:L_4x4, symbol device:L_Small
- removed U5: LM2596S-5, TO_SOT_Packages_SMD:TO-263-5_TabPin3, symbol dc-dc:LM2596S-5
- added C13, C15, C23, C31, C32, C9: 10uF, Capacitors_SMD:C_1206, symbol device:C_Small
- added D2: SS34, symbol device:D_Schottky_ALT
- added R29: 10K, symbol device:R_Small
- added R30: 1K, symbol device:R_Small
- added U10, U9: LD1117S50TR_SOT223, TO_SOT_Packages_SMD:SOT-223-3Lead_TabPin2, symbol regul:LD1117S50TR_SOT223
- added U5: SD6271LR, symbol SHOUDING:SD6271LR
- L1: value 33uH -> 4.7uH; footprint custom_inductors:L_4x4 -> (none)
- R8: value 1k -> 51K; footprint Resistors_SMD:R_0805 -> (none)
Connections:
- net +3V3: now also J3.1 (VBUS), L1.2, C9.2, U5.4 (EN), U5.5 (VCC)
- net +5V: now also C32.2, U10.2 (VO); no longer C16.2, L1.2, U6.3 (VI)
- net +5VA: now also C31.2, U9.2 (VO)
- net GND: now also R8.2, C13.1, C15.1, C23.1, C31.1, C32.1, C9.1, R30.2, U10.1 (GND), U5.2 (GND), U9.1 (GND); no longer C11.2, C14.1, C18.2, C27.2, R19.2, R20.2, R21.2, R22.2, U3.19 (AGND), U4.6 (OE), U4.8 (GND), U8.4 (V-)
- net at L1.1: now also D2.2 (A), U5.1 (LX)
- net +12V: no longer names the net of R8.1
- net +12V: now also U5.6 (OC)
- new net: C13.2, C15.2, C16.2, C23.2, D2.1 (K), R29.1, U10.3 (VI), U6.3 (VI), U9.3 (VI)
- new net: R29.2, R30.1, U5.3 (FB)
- new net GNDA: C11.2, C14.1, C18.2, C27.2, R19.2, R20.2, R21.2, R22.2, U3.19 (AGND), U4.6 (OE), U4.8 (GND), U8.4 (V-)
- no-connect marks 19 -> 18
Other:
- moved on the sheet: C16, C17, U6

Commit message: Pre-reroute
Parts:
- C18, C29, C30: footprint (none) -> Capacitors_SMD:CP_Elec_6.3x7.7
- C19, C22: footprint (none) -> Capacitors_SMD:C_1206
- C20, C21, C24, C25: footprint (none) -> Capacitors_SMD:C_0805
- D2: footprint (none) -> Diodes_SMD:D_SMA
- L1: footprint (none) -> custom_inductors:L_4x4
- R18, R19, R20, R21, R22, R23, R24, R25, R26, R27, R28, R29, R30, R8: footprint (none) -> Resistors_SMD:R_0805
- U10, U9: footprint TO_SOT_Packages_SMD:SOT-223-3Lead_TabPin2 -> TO_SOT_Packages_SMD:SOT-223-3_TabPin2
- U5: footprint (none) -> TO_SOT_Packages_SMD:SOT-23-6
- U8: footprint (none) -> Housings_SOIC:SOIC-8_3.9x4.9mm_Pitch1.27mm
Changed lines of the file:
@@
 F 0 "U8" H 13041 1746 50  0000 L CNN
 F 1 "TL072" H 13041 1655 50  0000 L CNN
-F 2 "" H 12700 1700 50  0001 C CNN
+F 2 "Housings_SOIC:SOIC-8_3.9x4.9mm_Pitch1.27mm" H 12700 1700 50  0001 C CNN
 F 3 "http://www.ti.com/lit/ds/symlink/tl071.pdf" H 12700 1700 50  0001 C CNN
 	1    12700 1700
@@
 F 0 "U8" H 13041 3346 50  0000 L CNN
 F 1 "TL072" H 13041 3255 50  0000 L CNN
-F 2 "" H 12700 3300 50  0001 C CNN
+F 2 "Housings_SOIC:SOIC-8_3.9x4.9mm_Pitch1.27mm" H 12700 3300 50  0001 C CNN
 F 3 "http://www.ti.com/lit/ds/symlink/tl071.pdf" H 12700 3300 50  0001 C CNN
 	2    12700 3300
@@
 F 0 "R18" H 10359 946 50  0000 L CNN
 F 1 "10K" H 10359 855 50  0000 L CNN
-F 2 "" H 10300 900 50  0001 C CNN
+F 2 "Resistors_SMD:R_0805" H 10300 900 50  0001 C CNN
 F 3 "~" H 10300 900 50  0001 C CNN
 	1    10300 900
@@
 F 0 "R19" H 10359 1346 50  0000 L CNN
 F 1 "10K" H 10359 1255 50  0000 L CNN
-F 2 "" H 10300 1300 50  0001 C CNN
+F 2 "Resistors_SMD:R_0805" H 10300 1300 50  0001 C CNN
 F 3 "~" H 10300 1300 50  0001 C CNN
 	1    10300 1300
@@
 F 0 "C18" H 10838 1346 50  0000 L CNN
 F 1 "100uF" H 10838 1255 50  0000 L CNN
-F 2 "" H 10750 1300 50  0001 C CNN
+F 2 "Capacitors_SMD:CP_Elec_6.3x7.7" H 10750 1300 50  0001 C CNN
 F 3 "~" H 10750 1300 50  0001 C CNN
 	1    10750 1300
@@
 F 0 "R20" H 10459 2146 50  0000 L CNN
 F 1 "2.2K" H 10459 2055 50  0000 L CNN
-F 2 "" H 10400 2100 50  0001 C CNN
+F 2 "Resistors_SMD:R_0805" H 10400 2100 50  0001 C CNN
 F 3 "~" H 10400 2100 50  0001 C CNN
 	1    10400 2100
@@
 F 0 "R22" H 10459 3346 50  0000 L CNN
 F 1 "2.2K" H 10459 3255 50  0000 L CNN
-F 2 "" H 10400 3300 50  0001 C CNN
+F 2 "Resistors_SMD:R_0805" H 10400 3300 50  0001 C CNN
 F 3 "~" H 10400 3300 50  0001 C CNN
 	1    10400 3300
@@
 F 0 "R21" H 10459 2746 50  0000 L CNN
 F 1 "2.2K" H 10459 2655 50  0000 L CNN
-F 2 "" H 10400 2700 50  0001 C CNN
+F 2 "Resistors_SMD:R_0805" H 10400 2700 50  0001 C CNN
 F 3 "~" H 10400 2700 50  0001 C CNN
 	1    10400 2700
@@
 F 0 "C20" V 10671 2400 50  0000 C CNN
 F 1 "1uF" V 10762 2400 50  0000 C CNN
-F 2 "" H 10900 2400 50  0001 C CNN
+F 2 "Capacitors_SMD:C_0805" H 10900 2400 50  0001 C CNN
 F 3 "~" H 10900 2400 50  0001 C CNN
 	1    10900 2400
@@
 F 0 "C21" V 10671 2850 50  0000 C CNN
 F 1 "1uF" V 10762 2850 50  0000 C CNN
-F 2 "" H 10900 2850 50  0001 C CNN
+F 2 "Capacitors_SMD:C_0805" H 10900 2850 50  0001 C CNN
 F 3 "~" H 10900 2850 50  0001 C CNN
 	1    10900 2850
@@
 F 0 "C19" V 10671 2000 50  0000 C CNN
 F 1 "10uF" V 10762 2000 50  0000 C CNN
-F 2 "" H 10900 2000 50  0001 C CNN
+F 2 "Capacitors_SMD:C_1206" H 10900 2000 50  0001 C CNN
 F 3 "~" H 10900 2000 50  0001 C CNN
 	1    10900 2000
@@
 F 0 "C22" V 10671 3200 50  0000 C CNN
 F 1 "10uF" V 10762 3200 50  0000 C CNN
-F 2 "" H 10900 3200 50  0001 C CNN
+F 2 "Capacitors_SMD:C_1206" H 10900 3200 50  0001 C CNN
 F 3 "~" H 10900 3200 50  0001 C CNN
 	1    10900 3200
@@
 F 0 "R24" V 10904 2400 50  0000 C CNN
 F 1 "51K" V 10995 2400 50  0000 C CNN
-F 2 "" H 11100 2400 50  0001 C CNN
+F 2 "Resistors_SMD:R_0805" H 11100 2400 50  0001 C CNN
 F 3 "~" H 11100 2400 50  0001 C CNN
 	1    11100 2400
@@
 F 0 "R25" V 10904 2850 50  0000 C CNN
 F 1 "51K" V 10995 2850 50  0000 C CNN
-F 2 "" H 11100 2850 50  0001 C CNN
+F 2 "Resistors_SMD:R_0805" H 11100 2850 50  0001 C CNN
 F 3 "~" H 11100 2850 50  0001 C CNN
 	1    11100 2850
@@
 F 0 "R23" V 10904 2000 50  0000 C CNN
 F 1 "6.2K" V 10995 2000 50  0000 C CNN
-F 2 "" H 11100 2000 50  0001 C CNN
+F 2 "Resistors_SMD:R_0805" H 11100 2000 50  0001 C CNN
 F 3 "~" H 11100 2000 50  0001 C CNN
 	1    11100 2000
@@
 F 0 "R26" V 10904 3200 50  0000 C CNN
 F 1 "6.2K" V 10995 3200 50  0000 C CNN
-F 2 "" H 11100 3200 50  0001 C CNN
+F 2 "Resistors_SMD:R_0805" H 11100 3200 50  0001 C CNN
 F 3 "~" H 11100 3200 50  0001 C CNN
 	1    11100 3200
@@
 F 0 "R27" V 12404 2450 50  0000 C CNN
 F 1 "160K" V 12500 2450 50  0000 C CNN
-F 2 "" H 12600 2450 50  0001 C CNN
+F 2 "Resistors_SMD:R_0805" H 12600 2450 50  0001 C CNN
 F 3 "~" H 12600 2450 50  0001 C CNN
 	1    12600 2450
@@
 F 0 "C24" V 12371 2750 50  0000 C CNN
 F 1 "270pF" V 12462 2750 50  0000 C CNN
-F 2 "" H 12600 2750 50  0001 C CNN
+F 2 "Capacitors_SMD:C_0805" H 12600 2750 50  0001 C CNN
 F 3 "~" H 12600 2750 50  0001 C CNN
 	1    12600 2750
@@
 F 0 "R28" V 12404 3850 50  0000 C CNN
 F 1 "160K" V 12500 3850 50  0000 C CNN
-F 2 "" H 12600 3850 50  0001 C CNN
+F 2 "Resistors_SMD:R_0805" H 12600 3850 50  0001 C CNN
 F 3 "~" H 12600 3850 50  0001 C CNN
 	1    12600 3850
@@
 F 0 "C25" V 12371 4150 50  0000 C CNN
 F 1 "270pF" V 12462 4150 50  0000 C CNN
-F 2 "" H 12600 4150 50  0001 C CNN
+F 2 "Capacitors_SMD:C_0805" H 12600 4150 50  0001 C CNN
 F 3 "~" H 12600 4150 50  0001 C CNN
 	1    12600 4150
@@
 F 0 "C29" V 13675 1700 50  0000 C CNN
 F 1 "100uF" V 13584 1700 50  0000 C CNN
-F 2 "" H 13450 1700 50  0001 C CNN
+F 2 "Capacitors_SMD:CP_Elec_6.3x7.7" H 13450 1700 50  0001 C CNN
 F 3 "~" H 13450 1700 50  0001 C CNN
 	1    13450 1700
@@
 F 0 "C30" V 13675 3300 50  0000 C CNN
 F 1 "100uF" V 13584 3300 50  0000 C CNN
-F 2 "" H 13450 3300 50  0001 C CNN
+F 2 "Capacitors_SMD:CP_Elec_6.3x7.7" H 13450 3300 50  0001 C CNN
 F 3 "~" H 13450 3300 50  0001 C CNN
 	1    13450 3300
@@
 F 0 "U5" H 6025 7725 50  0000 C CNN
 F 1 "SD6271LR" H 6025 7634 50  0000 C CNN
-F 2 "" H 5800 7000 50  0001 C CNN
+F 2 "TO_SOT_Packages_SMD:SOT-23-6" H 5800 7000 50  0001 C CNN
 F 3 "" H 5800 7000 50  0001 C CNN
 	1    5800 7000
@@
 F 0 "R8" H 5659 6846 50  0000 L CNN
 F 1 "51K" H 5659 6755 50  0000 L CNN
-F 2 "" H 5600 6800 50  0001 C CNN
+F 2 "Resistors_SMD:R_0805" H 5600 6800 50  0001 C CNN
 F 3 "~" H 5600 6800 50  0001 C CNN
 	1    5600 6800
@@
 F 0 "L1" V 5872 7250 50  0000 C CNN
 F 1 "4.7uH" V 5963 7250 50  0000 C CNN
-F 2 "" H 6050 7250 50  0001 C CNN
+F 2 "custom_inductors:L_4x4" H 6050 7250 50  0001 C CNN
 F 3 "~" H 6050 7250 50  0001 C CNN
 	1    6050 7250
@@
 F 0 "D2" H 7050 6484 50  0000 C CNN
 F 1 "SS34" H 7050 6575 50  0000 C CNN
-F 2 "" H 7050 6700 50  0001 C CNN
+F 2 "Diodes_SMD:D_SMA" H 7050 6700 50  0001 C CNN
 F 3 "~" H 7050 6700 50  0001 C CNN
 	1    7050 6700
@@
 F 0 "R29" H 7259 6846 50  0000 L CNN
 F 1 "10K" H 7259 6755 50  0000 L CNN
-F 2 "" H 7200 6800 50  0001 C CNN
+F 2 "Resistors_SMD:R_0805" H 7200 6800 50  0001 C CNN
 F 3 "~" H 7200 6800 50  0001 C CNN
 	1    7200 6800
@@
 F 0 "R30" H 7259 7146 50  0000 L CNN
 F 1 "1K" H 7259 7055 50  0000 L CNN
-F 2 "" H 7200 7100 50  0001 C CNN
+F 2 "Resistors_SMD:R_0805" H 7200 7100 50  0001 C CNN
 F 3 "~" H 7200 7100 50  0001 C CNN
 	1    7200 7100
@@
 F 0 "U10" H 8500 6450 50  0000 C CNN
 F 1 "LD1117S50TR_SOT223" H 8350 6851 50  0000 C CNN
-F 2 "TO_SOT_Packages_SMD:SOT-223-3Lead_TabPin2" H 8350 6900 50  0001 C CNN
+F 2 "TO_SOT_Packages_SMD:SOT-223-3_TabPin2" H 8350 6900 50  0001 C CNN
 F 3 "http://www.st.com/st-web-ui/static/active/en/resource/technical/document/datasheet/CD00000544.pdf" H 8450 6450 50  0001 C CNN
 	1    8350 6700
@@
 F 0 "U9" H 8350 6192 50  0000 C CNN
 F 1 "LD1117S50TR_SOT223" H 8350 6101 50  0000 C CNN
-F 2 "TO_SOT_Packages_SMD:SOT-223-3Lead_TabPin2" H 8350 6150 50  0001 C CNN
+F 2 "TO_SOT_Packages_SMD:SOT-223-3_TabPin2" H 8350 6150 50  0001 C CNN
 F 3 "http://www.st.com/st-web-ui/static/active/en/resource/technical/document/datasheet/CD00000544.pdf" H 8450 5700 50  0001 C CNN
 	1    8350 5950

Commit message: Analog stage
Parts:
- J6: footprint Connectors:PJ320E_3.5mm_Jack -> Boom Precision Elec PJ-307C:SWITCHCRAFT_35RAPC4BHN2
Connections:
- net GNDA is gone; now on net GND: C11.2, C14.1, C18.2, C27.2, R19.2, R20.2, R21.2, R22.2, U3.19 (AGND), U4.6 (OE), U4.8 (GND), U8.4 (V-)
- net +3V3: no longer C9.2, J3.1 (VBUS), L1.2, U5.4 (EN), U5.5 (VCC)
- net +5VA: now also U8.8 (V+)
- net GND: now also U8.4 (V-)
- new net VBUS: C9.2, J3.1 (VBUS), L1.2, U5.4 (EN), U5.5 (VCC)
Other:
- moved on the sheet: C25, R28
Changed lines of the file:
@@
 F 0 "J6" H 9976 9025 50  0000 C CNN
 F 1 "Audio-Jack-3" H 9976 8934 50  0000 C CNN
-F 2 "Connectors:PJ320E_3.5mm_Jack" H 10250 8800 50  0001 C CNN
+F 2 "Boom Precision Elec PJ-307C:SWITCHCRAFT_35RAPC4BHN2" H 10250 8800 50  0001 C CNN
 F 3 "~" H 10250 8800 50  0001 C CNN
 	1    10000 8700
@@
 L device:R_Small R28
 U 1 1 5D2448FB
-P 12600 3850
-F 0 "R28" V 12404 3850 50  0000 C CNN
-F 1 "160K" V 12500 3850 50  0000 C CNN
-F 2 "Resistors_SMD:R_0805" H 12600 3850 50  0001 C CNN
-F 3 "~" H 12600 3850 50  0001 C CNN
-	1    12600 3850
+P 12600 4100
+F 0 "R28" V 12404 4100 50  0000 C CNN
+F 1 "160K" V 12500 4100 50  0000 C CNN
+F 2 "Resistors_SMD:R_0805" H 12600 4100 50  0001 C CNN
+F 3 "~" H 12600 4100 50  0001 C CNN
+	1    12600 4100
 	0    1    1    0
 $EndComp
@@
 L device:C_Small C25
 U 1 1 5D244A15
-P 12600 4150
-F 0 "C25" V 12371 4150 50  0000 C CNN
-F 1 "270pF" V 12462 4150 50  0000 C CNN
-F 2 "Capacitors_SMD:C_0805" H 12600 4150 50  0001 C CNN
-F 3 "~" H 12600 4150 50  0001 C CNN
-	1    12600 4150
-	0    1    1    0
-$EndComp
-Wire Wire Line
-	12400 3400 12400 3850
-Wire Wire Line
-	12400 3850 12500 3850
-Connection ~ 12400 3400
-Wire Wire Line
-	12400 3850 12400 4150
-Wire Wire Line
-	12400 4150 12500 4150
-Connection ~ 12400 3850
-Wire Wire Line
-	12700 4150 13000 4150
-Wire Wire Line
-	13000 4150 13000 3850
-Wire Wire Line
-	12700 3850 13000 3850
-Connection ~ 13000 3850
-Wire Wire Line
-	13000 3850 13000 3300
+P 12600 4400
+F 0 "C25" V 12371 4400 50  0000 C CNN
+F 1 "270pF" V 12462 4400 50  0000 C CNN
+F 2 "Capacitors_SMD:C_0805" H 12600 4400 50  0001 C CNN
+F 3 "~" H 12600 4400 50  0001 C CNN
+	1    12600 4400
+	0    1    1    0
+$EndComp
+Wire Wire Line
+	12400 4100 12500 4100
+Wire Wire Line
+	12400 4100 12400 4400
+Wire Wire Line
+	12400 4400 12500 4400
+Connection ~ 12400 4100
+Wire Wire Line
+	12700 4400 13000 4400
+Wire Wire Line
+	13000 4400 13000 4100
+Wire Wire Line
+	12700 4100 13000 4100
+Connection ~ 13000 4100
 Wire Wire Line
 	11400 1800 12400 1800
@@
 Wire Wire Line
 	13000 3300 13350 3300
-Connection ~ 13000 3300
 Wire Wire Line
 	13000 1700 13350 1700
@@
 Wire Notes Line
 	4450 7600 11200 7600
-$Comp
-L power:VCC #PWR033
-U 1 1 5D186322
-P 4950 8400
-F 0 "#PWR033" H 4950 8250 50  0001 C CNN
-F 1 "VCC" H 4967 8573 50  0000 C CNN
-F 2 "" H 4950 8400 50  0001 C CNN
-F 3 "" H 4950 8400 50  0001 C CNN
-	1    4950 8400
-	1    0    0    -1
-$EndComp
 Wire Wire Line
 	9550 6700 9550 7200
@@
 	1    6050 7250
 	0    1    1    0
-$EndComp
-$Comp
-L power:VCC #PWR034
-U 1 1 5D1A5741
-P 5100 6500
-F 0 "#PWR034" H 5100 6350 50  0001 C CNN
-F 1 "VCC" H 5117 6673 50  0000 C CNN
-F 2 "" H 5100 6500 50  0001 C CNN
-F 3 "" H 5100 6500 50  0001 C CNN
-	1    5100 6500
-	1    0    0    -1
 $EndComp
 Wire Wire Line
@@
 Wire Wire Line
 	5100 6500 5100 6650
-Connection ~ 5100 6500
 $Comp
 L power:GND #PWR035
@@
 Wire Wire Line
 	7750 6700 7850 6700
+$Comp
+L power:VBUS #PWR0101
+U 1 1 5D31B3CA
+P 4950 8400
+F 0 "#PWR0101" H 4950 8250 50  0001 C CNN
+F 1 "VBUS" H 4965 8573 50  0000 C CNN
+F 2 "" H 4950 8400 50  0001 C CNN
+F 3 "" H 4950 8400 50  0001 C CNN
+	1    4950 8400
+	1    0    0    -1
+$EndComp
+$Comp
+L power:VBUS #PWR0102
+U 1 1 5D31B9A5
+P 5100 6500
+F 0 "#PWR0102" H 5100 6350 50  0001 C CNN
+F 1 "VBUS" H 5115 6673 50  0000 C CNN
+F 2 "" H 5100 6500 50  0001 C CNN
+F 3 "" H 5100 6500 50  0001 C CNN
+	1    5100 6500
+	1    0    0    -1
+$EndComp
+Connection ~ 5100 6500
+$Comp
+L power:GND #PWR0103
+U 1 1 5D31D3AE
+P 10900 6800
+F 0 "#PWR0103" H 10900 6550 50  0001 C CNN
+F 1 "GND" H 10905 6627 50  0000 C CNN
+F 2 "" H 10900 6800 50  0001 C CNN
+F 3 "" H 10900 6800 50  0001 C CNN
+	1    10900 6800
+	1    0    0    -1
+$EndComp
+$Comp
+L power:GNDA #PWR0104
+U 1 1 5D31D4A2
+P 10550 6800
+F 0 "#PWR0104" H 10550 6550 50  0001 C CNN
+F 1 "GNDA" H 10555 6627 50  0000 C CNN
+F 2 "" H 10550 6800 50  0001 C CNN
+F 3 "" H 10550 6800 50  0001 C CNN
+	1    10550 6800
+	1    0    0    -1
+$EndComp
+Wire Wire Line
+	10550 6800 10900 6800
+$Comp
+L power:+5VA #PWR0105
+U 1 1 5D32A00D
+P 12600 3000
+F 0 "#PWR0105" H 12600 2850 50  0001 C CNN
+F 1 "+5VA" H 12615 3173 50  0000 C CNN
+F 2 "" H 12600 3000 50  0001 C CNN
+F 3 "" H 12600 3000 50  0001 C CNN
+	1    12600 3000
+	1    0    0    -1
+$EndComp
+Wire Wire Line
+	13000 3300 13000 4100
+Connection ~ 13000 3300
+Wire Wire Line
+	12400 3400 12400 4100
+Connection ~ 12400 3400
+$Comp
+L power:GNDA #PWR?
+U 1 1 5D3474C0
+P 12600 3600
+F 0 "#PWR?" H 12600 3350 50  0001 C CNN
+F 1 "GNDA" H 12605 3427 50  0000 C CNN
+F 2 "" H 12600 3600 50  0001 C CNN
+F 3 "" H 12600 3600 50  0001 C CNN
+	1    12600 3600
+	1    0    0    -1
+$EndComp
 $EndSCHEMATC

Commit message: Route complete
Connections:
- net 6.6VBOOST: now reaches C13.2, C15.2, C16.2, C23.2, D2.1 (K), R29.1, U10.3 (VI), U6.3 (VI), U9.3 (VI)
Other:
- moved on the sheet: C13, C15, C16, C17, C23, C31, C32, C9, D2, L1, R29, R30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
