File: Schematic/YM2612_MIDI_SMD/YM2612_MIDI_SMD.sch (KiCad schematic (older format))
At the start: 107 parts, among them J1 DIN-5_180, J2 TP_GND, J3 USB_B, J5 ICSP, J6 Audio-Jack-3, J7 Micro_SD_Card, SW1 Rotary_Encoder_Switch, SW10 SW_Push_Dual, SW2 SW_Push_Dual, SW3 SW_Push_Dual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

Commit message: Amend PSG resistors
Parts:
- R21: value 2.2K -> 1.3K
- R24, R25: value 51K -> 150K
Changed lines of the file:
@@
 P 10400 2700
 F 0 "R21" H 10459 2746 50  0000 L CNN
-F 1 "2.2K" H 10459 2655 50  0000 L CNN
+F 1 "1.3K" H 10459 2655 50  0000 L CNN
 F 2 "Resistors_SMD:R_0805" H 10400 2700 50  0001 C CNN
 F 3 "~" H 10400 2700 50  0001 C CNN
@@
 P 11100 2400
 F 0 "R24" V 10904 2400 50  0000 C CNN
-F 1 "51K" V 10995 2400 50  0000 C CNN
+F 1 "150K" V 10995 2400 50  0000 C CNN
 F 2 "Resistors_SMD:R_0805" H 11100 2400 50  0001 C CNN
 F 3 "~" H 11100 2400 50  0001 C CNN
@@
 P 11100 2850
 F 0 "R25" V 10904 2850 50  0000 C CNN
-F 1 "51K" V 10995 2850 50  0000 C CNN
+F 1 "150K" V 10995 2850 50  0000 C CNN
 F 2 "Resistors_SMD:R_0805" H 11100 2850 50  0001 C CNN
 F 3 "~" H 11100 2850 50  0001 C CNN

Commit message: Adjusted resistor values
Parts:
- added MP1: GRAPHIC, art:logo_1, symbol TPA3122D2:GRAPHIC
- added MP2: GRAPHIC, art:logo_2, symbol TPA3122D2:GRAPHIC
- added MP3: GRAPHIC, art:logo_3, symbol TPA3122D2:GRAPHIC
Changed lines of the file:
@@
 	8200 6700 8300 6700
 Connection ~ 8300 6700
+$Comp
+L TPA3122D2:GRAPHIC MP1
+U 1 1 5D20DA8B
+P 11300 10050
+F 0 "MP1" H 11300 10249 20  0000 C CNN
+F 1 "GRAPHIC" H 11300 10206 20  0000 C CNN
+F 2 "art:logo_1" H 11300 10131 60  0000 C CNN
+F 3 "" H 11300 10050 60  0000 C CNN
+	1    11300 10050
+	1    0    0    -1
+$EndComp
+$Comp
+L TPA3122D2:GRAPHIC MP2
+U 1 1 5D20E0BB
+P 11300 10200
+F 0 "MP2" H 11300 10399 20  0000 C CNN
+F 1 "GRAPHIC" H 11300 10356 20  0000 C CNN
+F 2 "art:logo_2" H 11300 10281 60  0000 C CNN
+F 3 "" H 11300 10200 60  0000 C CNN
+	1    11300 10200
+	1    0    0    -1
+$EndComp
+$Comp
+L TPA3122D2:GRAPHIC MP3
+U 1 1 5D20E1B3
+P 11300 10350
+F 0 "MP3" H 11300 10549 20  0000 C CNN
+F 1 "GRAPHIC" H 11300 10506 20  0000 C CNN
+F 2 "art:logo_3" H 11300 10431 60  0000 C CNN
+F 3 "" H 11300 10350 60  0000 C CNN
+	1    11300 10350
+	1    0    0    -1
+$EndComp
 $EndSCHEMATC

Commit message: New boost circuit
Parts:
- removed U5: SD6271LR, TO_SOT_Packages_SMD:SOT-23-6, symbol SHOUDING:SD6271LR
- added C33: 10uF, Capacitors_SMD:C_1206, symbol device:C_Small
- added U5: LM2733XMF, TO_SOT_Packages_SMD:SOT-23-5, symbol dc-dc:LM2733XMF
- C13: value 10uF -> 220pF; footprint Capacitors_SMD:C_1206 -> Capacitors_SMD:C_0603
- C6: footprint Capacitors_SMD:C_1206 -> Capacitors_SMD:C_0805
- L1: value 4.7uH -> 10uH
- R29: value 10K -> 12K
- R30: value 1K -> 51K
Connections:
- net GND: now also C9.2, R29.1, C33.2, U5.2 (GND); no longer C13.1, C9.1, J3.5 (Shield), R30.2, R8.2
- net VBUS: now also C9.1, R8.1, U5.5 (VIN); no longer C9.2
- net at D2.2 (A), L1.1: now also U5.1 (SW)
- net at R29.2: now also C13.2, R30.2, U5.3 (FB); no longer R30.1
- net 6.6VBOOST renamed VBOOST
- net VBOOST: now also C13.1, R30.1, C33.1; no longer C13.2, R29.1
- new net: R8.2, U5.4 (EN)
- no-connect marks 18 -> 19

Commit message: Amplifier notations
Other:
- note added: "YM3438 Change:\nR23, R26 51K"
- note added: "YM3438 Remove:\nR20\nR22"
Changed lines of the file:
@@
 	4900 6500 5150 6500
 NoConn ~ 4550 9000
+Text Notes 10000 4050 0    50   ~ 0
+YM3438 Remove:\nR20\nR22
+Text Notes 10000 4350 0    50   ~ 0
+YM3438 Change:\nR23, R26 51K
 $EndSCHEMATC
